Commit message: mm

File: spider_description/urdf/spider_description_1.xacro (robot description, xacro)
@@ -8,7 +8,7 @@
   <link name="base_link">
     <inertial>
-      <origin xyz="0.0513553543804905 -0.00355010292388771 0.0158371951293718" rpy="0 0 0" />
-      <mass value="0.206587820695411" />
-      <inertia ixx="9.18101041743378E-05" ixy="-1.1096915717602E-06" ixz="-2.07334737671996E-08" iyy="0.000621158029436724" iyz="3.17880975410803E-08" izz="0.000699601373790156" />
+      <origin xyz="0.0419124697856288 0.0129912705123136 -0.00194512919498489" rpy="0 0 0" />
+      <mass value="0.206593361987693" />
+      <inertia ixx="0.000100835459421752" ixy="3.3190326442876E-07" ixz="6.85143109069958E-05" iyy="0.000699628428109392" iyz="-7.47632670675628E-08" izz="0.000612159753876248" />
     </inertial>
     <visual>
@@ -30,7 +30,7 @@
   <link name="RL1_coxa">
     <inertial>
-      <origin xyz="-0.00349163844394274 0.017230005966643 0.0244390511872048" rpy="0 0 0" />
-      <mass value="0.0118214531865819" />
-      <inertia ixx="1.54720054808557E-06" ixy="-3.57557713352019E-08" ixz="-4.02762646820984E-08" iyy="1.03828147386784E-06" iyz="-8.80078006023742E-10" izz="1.47258288978444E-06" />
+      <origin xyz="-0.00349163991648843 0.0172300072694273 0.024439051068252" rpy="0 0 0" />
+      <mass value="0.0118214563639757" />
+      <inertia ixx="1.54720113656629E-06" ixy="-3.57556957341545E-08" ixz="-4.0276165283765E-08" iyy="1.03828170219183E-06" iyz="-8.80235914490984E-10" izz="1.47258336300693E-06" />
     </inertial>
     <visual>
@@ -51,5 +51,5 @@
   </link>
   <joint name="joint1_coxa" type="continuous">
-    <origin xyz="0.14757063197026 -0.0470606865446389 0.00464999999999999" rpy="1.5707963267949 0 0.216963279781621" />
+    <origin xyz="0.143023923046985 -0.028827601978856 0.00180390069504784" rpy="1.5707963267949 0 0.456646809528589" />
     <parent link="base_link" />
     <child link="RL1_coxa" />
@@ -58,7 +58,7 @@
   <link name="RL1_fumer">
     <inertial>
-      <origin xyz="-0.0264233888332985 -1.38777878078145E-17 -0.00234030420177742" rpy="0 0 0" />
-      <mass value="0.00732061922605987" />
-      <inertia ixx="1.66034801156123E-06" ixy="-7.94093388050907E-22" ixz="-1.49987503139404E-09" iyy="3.3348950865199E-06" iyz="1.28978137012331E-21" izz="1.8515397312667E-06" />
+      <origin xyz="-0.0264233888332986 6.93889390390723E-18 -0.00234030420177805" rpy="0 0 0" />
+      <mass value="0.00732061922605988" />
+      <inertia ixx="1.66034801156124E-06" ixy="1.00585162486448E-21" ixz="-1.49987503139991E-09" iyy="3.33489508651991E-06" iyz="1.04555629426703E-21" izz="1.85153973126671E-06" />
     </inertial>
     <visual>
@@ -79,5 +79,5 @@
   </link>
   <joint name="joint1_fumer" type="continuous">
-    <origin xyz="-0.00591979008225604 0.0221000000000001 0.0268552804003611" rpy="-1.98602850950399 1.00791673675336 1.213911849099" />
+    <origin xyz="-0.00591979008225604 0.0221000000000001 0.026855280400361" rpy="-2.03537963970565 1.06963032129347 1.15667679281028" />
     <parent link="RL1_coxa" />
     <child link="RL1_fumer" />
@@ -86,7 +86,7 @@
   <link name="RL1_tibia">
     <inertial>
-      <origin xyz="0.00260154713513186 -0.0130975375024425 0.000727426073779153" rpy="0 0 0" />
-      <mass value="0.013123891605465" />
-      <inertia ixx="4.2299662226924E-06" ixy="1.19149413513681E-07" ixz="-1.17548988409946E-08" iyy="7.82194147309099E-07" iyz="-2.83284559215829E-07" izz="4.42455942176531E-06" />
+      <origin xyz="0.00260154719028149 -0.013097537565338 0.000727426101389261" rpy="0 0 0" />
+      <mass value="0.0131238915671885" />
+      <inertia ixx="4.22996621859555E-06" ixy="1.19149405996142E-07" ixz="-1.17548949137053E-08" iyy="7.82194141970863E-07" iyz="-2.83284562385563E-07" izz="4.4245594105805E-06" />
     </inertial>
     <visual>
@@ -107,5 +107,5 @@
   </link>
   <joint name="joint1_tibia" type="continuous">
-    <origin xyz="-0.055 0 0" rpy="3.14159265358979 1.35383304701328 0.527393489709591" />
+    <origin xyz="-0.055 0 0" rpy="3.14159265358979 1.35383304701328 0.455416754848752" />
     <parent link="RL1_fumer" />
     <child link="RL1_tibia" />
@@ -114,7 +114,7 @@
   <link name="RL2_coxa">
     <inertial>
-      <origin xyz="-0.00137410211994941 0.017230005966643 0.024648947347057" rpy="0 0 0" />
-      <mass value="0.0118214531865819" />
-      <inertia ixx="1.53973619894474E-06" ixy="-3.56987341340023E-08" ixz="-4.6080725279413E-08" iyy="1.03828147386784E-06" iyz="2.20229478084549E-09" izz="1.48004723892527E-06" />
+      <origin xyz="-0.00137410359807341 0.0172300072704422 0.0246489473554496" rpy="0 0 0" />
+      <mass value="0.0118214563661804" />
+      <inertia ixx="1.53973680405956E-06" ixy="-3.56986723887601E-08" ixz="-4.6080637183373E-08" iyy="1.0382817023383E-06" iyz="2.2021308274049E-09" izz="1.4800476962292E-06" />
     </inertial>
     <visual>
@@ -135,5 +135,5 @@
   </link>
   <joint name="joint2_coxa" type="continuous">
-    <origin xyz="0.0870706319702602 -0.0470606865446389 0.00464999999999997" rpy="1.5707963267949 0 0.130741621531395" />
+    <origin xyz="0.0830253362173002 -0.0366006051591393 0.00180390069504788" rpy="1.5707963267949 0 0.371215936961481" />
     <parent link="base_link" />
     <child link="RL2_coxa" />
@@ -142,7 +142,7 @@
   <link name="RL2_fumer">
     <inertial>
-      <origin xyz="-0.0264233888332987 6.24500451351651E-17 0.0581596957982228" rpy="0 0 0" />
+      <origin xyz="-0.0264233888332985 0 -0.00234030420177726" rpy="0 0 0" />
       <mass value="0.00732061922605988" />
-      <inertia ixx="1.66034801156124E-06" ixy="5.82335151237331E-22" ixz="-1.49987503139389E-09" iyy="3.33489508651991E-06" iyz="3.18774728562622E-22" izz="1.85153973126671E-06" />
+      <inertia ixx="1.66034801156124E-06" ixy="3.70576914423756E-22" ixz="-1.49987503139454E-09" iyy="3.33489508651991E-06" iyz="-2.5146290621612E-22" izz="1.85153973126671E-06" />
     </inertial>
     <visual>
@@ -163,5 +163,5 @@
   </link>
   <joint name="joint2_fumer" type="continuous">
-    <origin xyz="0.0563985011948722 0.0221000000000001 0.0351526537116618" rpy="-1.82795682053227 1.0325993659782 1.3487143343647" />
+    <origin xyz="-0.00358516044020296 0.0220999999999999 0.0272653007432159" rpy="-1.84005724604345 1.0586197588623 1.33473036772911" />
     <parent link="RL2_coxa" />
     <child link="RL2_fumer" />
@@ -170,7 +170,7 @@
   <link name="RL2_tibia">
     <inertial>
-      <origin xyz="-0.0562495143524853 -0.0130839593275274 -0.00677615060162512" rpy="0 0 0" />
-      <mass value="0.013123891605465" />
-      <inertia ixx="4.23019150195768E-06" ixy="7.84253861591576E-08" ixz="1.01977946227722E-09" iyy="7.65338483748999E-07" iyz="-1.6371410447347E-07" izz="4.44118980606013E-06" />
+      <origin xyz="0.00373414734956586 -0.0130839594099826 0.00111120240408577" rpy="0 0 0" />
+      <mass value="0.0131238915536145" />
+      <inertia ixx="4.23019149640981E-06" ixy="7.84253770640042E-08" ixz="1.01978479704144E-09" iyy="7.6533847696787E-07" iyz="-1.63714108486507E-07" izz="4.44118979210614E-06" />
     </inertial>
     <visual>
@@ -191,5 +191,5 @@
   </link>
   <joint name="joint2_tibia" type="continuous">
-    <origin xyz="-0.055 0 0" rpy="-3.14159265358979 1.4400547052635 0.491910301591065" />
+    <origin xyz="-0.055 0 0" rpy="-3.14159265358979 1.4400547052635 0.436973540292822" />
     <parent link="RL2_fumer" />
     <child link="RL2_tibia" />
@@ -198,7 +198,7 @@
   <link name="RL3_coxa">
     <inertial>
-      <origin xyz="0.00349358134474833 0.017230005966643 0.0244387735236787" rpy="0 0 0" />
-      <mass value="0.0118214531865818" />
-      <inertia ixx="1.51968642178633E-06" ixy="-3.45709794269535E-08" ixz="-5.40202742068447E-08" iyy="1.03828147386784E-06" iyz="9.17044723735258E-09" izz="1.50009701608367E-06" />
+      <origin xyz="0.00349358017075859 0.01723000702548 0.0244387737829021" rpy="0 0 0" />
+      <mass value="0.0118214556819711" />
+      <inertia ixx="1.51968692035686E-06" ixy="-3.45709549158988E-08" ixz="-5.40202304528258E-08" iyy="1.03828165876939E-06" iyz="9.17031077224167E-09" izz="1.50009735512406E-06" />
     </inertial>
     <visual>
@@ -219,5 +219,5 @@
   </link>
   <joint name="joint3_coxa" type="continuous">
-    <origin xyz="0.0265706319702601 -0.0470606865446388 0.00464999999999998" rpy="1.5707963267949 0 -0.0669380319605713" />
+    <origin xyz="0.0230267493876147 -0.0443736083394228 0.00180390069504786" rpy="1.5707963267949 0 0.115999004572643" />
     <parent link="base_link" />
     <child link="RL3_coxa" />
@@ -226,7 +226,7 @@
   <link name="RL3_fumer">
     <inertial>
-      <origin xyz="-0.0264233888332993 -3.12250225675825E-16 0.118659695798224" rpy="0 0 0" />
+      <origin xyz="-0.0190060888231168 -0.0093450118645113 -0.00493699671842929" rpy="0 0 0" />
       <mass value="0.00732061922605988" />
-      <inertia ixx="1.66034801156124E-06" ixy="-1.05879118406788E-22" ixz="-1.49987503139562E-09" iyy="3.33489508651991E-06" iyz="-7.61987364388377E-23" izz="1.85153973126671E-06" />
+      <inertia ixx="1.66034801156124E-06" ixy="-8.470329472543E-22" ixz="-1.4998750313965E-09" iyy="3.33489508651991E-06" iyz="-6.61744490042422E-23" izz="1.85153973126671E-06" />
     </inertial>
     <visual>
@@ -247,5 +247,5 @@
   </link>
   <joint name="joint3_fumer" type="continuous">
-    <origin xyz="0.122568440358491 0.0221000000000001 0.0193449587253901" rpy="-1.43751480215154 1.04333153380391 1.6861356410289" />
+    <origin xyz="-0.000624989213601535 0.0103198993706474 0.0294985850073072" rpy="-1.43474773528477 1.05506840370706 1.68932703577979" />
     <parent link="RL3_coxa" />
     <child link="RL3_fumer" />
@@ -254,7 +254,7 @@
   <link name="RL3_tibia">
     <inertial>
-      <origin xyz="-0.118005534421714 -0.0130894519462948 0.00839605198202775" rpy="0 0 0" />
-      <mass value="0.013123891605465" />
-      <inertia ixx="4.23878065273637E-06" ixy="4.20082265127764E-08" ixz="4.18757931219035E-08" iyy="7.691544615372E-07" iyz="-2.12494160023349E-07" izz="4.42878467749324E-06" />
+      <origin xyz="0.00531436167769063 -0.0130894520266102 0.000128909648472023" rpy="0 0 0" />
+      <mass value="0.013123891554142" />
+      <inertia ixx="4.23878064857726E-06" ixy="4.20082179122996E-08" ixz="4.18757972044376E-08" iyy="7.69154455506806E-07" iyz="-2.12494162555612E-07" izz="4.42878466326275E-06" />
     </inertial>
     <visual>
@@ -275,14 +275,14 @@
   </link>
   <joint name="joint3_tibia" type="continuous">
-    <origin xyz="-0.055 0 0" rpy="0 1.50385829483433 -2.63968666156776" />
+    <origin xyz="-0.0475826999898183 -0.0093450118645113 0" rpy="0 1.50385829483433 -2.6917648290032" />
     <parent link="RL3_fumer" />
     <child link="RL3_tibia" />
-    <axis xyz="0.997760486341758 0 -0.0668880549504799" />
+    <axis xyz="0.997760486341758 0 -0.0668880549504796" />
   </joint>
   <link name="RL4_coxa">
     <inertial>
-      <origin xyz="0.000221643372700031 0.0172339889705058 0.0247738629223978" rpy="0 0 0" />
-      <mass value="0.011831113051677" />
-      <inertia ixx="1.51589381883954E-06" ixy="3.36933681099745E-08" ixz="5.44221588671393E-08" iyy="1.03946591481982E-06" iyz="1.04055511028782E-08" izz="1.50574484630922E-06" />
+      <origin xyz="0.000221643431956145 0.0172339886263365 0.024773862822896" rpy="0 0 0" />
+      <mass value="0.0118311142541974" />
+      <inertia ixx="1.51589405750511E-06" ixy="3.36933854050161E-08" ixz="5.44221416465647E-08" iyy="1.03946598429508E-06" iyz="1.04056213225627E-08" izz="1.50574501931213E-06" />
     </inertial>
     <visual>
@@ -303,5 +303,5 @@
   </link>
   <joint name="joint4_coxa" type="continuous">
-    <origin xyz="-0.0339293680297398 -0.0470606865446389 0.00465" rpy="1.5707963267949 0 0.105302517917499" />
+    <origin xyz="-0.0369718374420689 -0.0521466115197065 0.00180390069504695" rpy="1.5707963267949 0 0.279272825129561" />
     <parent link="base_link" />
     <child link="RL4_coxa" />
@@ -310,7 +310,7 @@
   <link name="RL4_fumer">
     <inertial>
-      <origin xyz="-0.0264233888332989 1.38777878078145E-17 -0.176940304201777" rpy="0 0 0" />
-      <mass value="0.00732061922605987" />
-      <inertia ixx="1.66034801156123E-06" ixy="5.29395592033938E-22" ixz="-1.49987503139488E-09" iyy="3.3348950865199E-06" iyz="1.40101077504865E-22" izz="1.85153973126671E-06" />
+      <origin xyz="-0.0264233888332986 -1.38777878078145E-17 0.00455969579822089" rpy="0 0 0" />
+      <mass value="0.00732061922605989" />
+      <inertia ixx="1.66034801156124E-06" ixy="-1.11173074327127E-21" ixz="-1.49987503139615E-09" iyy="3.33489508651992E-06" iyz="-8.73502726855997E-22" izz="1.85153973126671E-06" />
     </inertial>
     <visual>
@@ -331,5 +331,5 @@
   </link>
   <joint name="joint4_fumer" type="continuous">
-    <origin xyz="0.177604166796266 0.0221000000000001 0.0464247771842149" rpy="1.3624761407313 1.03768167086435 1.39071609018261" />
+    <origin xyz="-0.00289047043580869 0.0221000000000014 0.0273476723078892" rpy="1.34757833958992 1.0760490052699 1.37361152936902" />
     <parent link="RL4_coxa" />
     <child link="RL4_fumer" />
@@ -338,7 +338,7 @@
   <link name="RL4_tibia">
     <inertial>
-      <origin xyz="-0.175875204861774 -0.0124119057129757 -0.0227969872954879" rpy="0 0 0" />
-      <mass value="0.013123891605465" />
-      <inertia ixx="4.23942335897909E-06" ixy="1.02033754178209E-07" ixz="-4.08467258993426E-09" iyy="1.36774622886964E-06" iyz="-1.36758688607792E-06" izz="3.8295502039181E-06" />
+      <origin xyz="0.0046194323285307 -0.0124119057556658 -0.00371988245181533" rpy="0 0 0" />
+      <mass value="0.0131238915753325" />
+      <inertia ixx="4.23942335586469E-06" ixy="1.02033759025192E-07" ixz="-4.08466826831512E-09" iyy="1.36774622353105E-06" iyz="-1.36758688276913E-06" izz="3.82955019670378E-06" />
     </inertial>
     <visual>
@@ -359,5 +359,5 @@
   </link>
   <joint name="joint4_tibia" type="continuous">
-    <origin xyz="-0.055 0 0" rpy="0 -1.4654938088774 -0.864064197891256" />
+    <origin xyz="-0.0550000000000001 0 0" rpy="0 -1.4654938088774 -0.809353512947539" />
     <parent link="RL4_fumer" />
     <child link="RL4_tibia" />
@@ -366,7 +366,7 @@
   <link name="LL1_coxa">
     <inertial>
-      <origin xyz="0.0170998828634738 0.0172339889705059 -0.0179272813314759" rpy="0 0 0" />
-      <mass value="0.011831113051677" />
-      <inertia ixx="1.45656947113537E-06" ixy="-1.69226594240046E-08" ixz="6.66890699376806E-09" iyy="1.03946591481982E-06" iyz="-3.09377139809669E-08" izz="1.56506919401288E-06" />
+      <origin xyz="0.0170998824043466 0.0172339901017211 -0.017927284271033" rpy="0 0 0" />
+      <mass value="0.0118311172441887" />
+      <inertia ixx="1.45657003099262E-06" ixy="-1.69225042702206E-08" ixz="6.66881674443564E-09" iyy="1.03946612492756E-06" iyz="-3.09376104608946E-08" izz="1.5650694795515E-06" />
     </inertial>
     <visual>
@@ -387,5 +387,5 @@
   </link>
   <joint name="joint5_coxa" type="continuous">
-    <origin xyz="0.14757063197026 0.0399393134553611 0.00465000000000003" rpy="1.5707963267949 0 0.876029873391859" />
+    <origin xyz="0.121433238114814 0.0561023239846096 0.00180390069504789" rpy="1.5707963267949 0 0.779171496523206" />
     <parent link="base_link" />
     <child link="LL1_coxa" />
@@ -394,7 +394,7 @@
   <link name="LL1_fumer">
     <inertial>
-      <origin xyz="-0.0264233888332986 0 0.00455969579822271" rpy="0 0 0" />
-      <mass value="0.00732061922605989" />
-      <inertia ixx="1.66034801156124E-06" ixy="5.29395592033938E-23" ixz="-1.49987503139556E-09" iyy="3.33489508651991E-06" iyz="1.7570350186392E-21" izz="1.85153973126671E-06" />
+      <origin xyz="-0.0264233888332985 0 0.00455969579822237" rpy="0 0 0" />
+      <mass value="0.00732061922605988" />
+      <inertia ixx="1.66034801156124E-06" ixy="5.29395592033938E-22" ixz="-1.49987503139699E-09" iyy="3.33489508651991E-06" iyz="-4.2351647362715E-22" izz="1.85153973126671E-06" />
     </inertial>
     <visual>
@@ -415,5 +415,5 @@
   </link>
   <joint name="joint5_fumer" type="continuous">
-    <origin xyz="0.0211255891188233 0.0221 -0.0176056662578457" rpy="-2.74678119264294 -0.58768354984189 2.49709435666674" />
+    <origin xyz="0.0211255891188228 0.0221 -0.0176056662578466" rpy="-2.73801909944616 -0.582101669425183 2.48122445090949" />
     <parent link="LL1_coxa" />
     <child link="LL1_fumer" />
@@ -422,7 +422,7 @@
   <link name="LL1_tibia">
     <inertial>
-      <origin xyz="-0.00279894261734365 -0.0130976424430121 -0.00313843380108422" rpy="0 0 0" />
-      <mass value="0.013123891605465" />
-      <inertia ixx="4.36602526509336E-06" ixy="-2.59110649699593E-07" ixz="-7.85274951562141E-08" iyy="7.97432607148881E-07" iyz="2.87128236854985E-07" izz="4.27326191952455E-06" />
+      <origin xyz="-0.00279894329842953 -0.0130976389443435 -0.00313843570289792" rpy="0 0 0" />
+      <mass value="0.0131238945399001" />
+      <inertia ixx="4.36602557276728E-06" ixy="-2.59110541265302E-07" ixz="-7.85276269962679E-08" iyy="7.97432719732035E-07" iyz="2.87128419374741E-07" izz="4.27326198471528E-06" />
     </inertial>
     <visual>
@@ -443,14 +443,14 @@
   </link>
   <joint name="joint5_tibia" type="continuous">
-    <origin xyz="-0.0549999999999999 0 0" rpy="3.14159265358979 0.694766453403041 2.59196218761899" />
+    <origin xyz="-0.0549999999999999 0 0" rpy="-3.14159265358979 0.69476645340304 2.60363290009658" />
     <parent link="LL1_fumer" />
     <child link="LL1_tibia" />
-    <axis xyz="0.640206045739847 0 0.768203240684487" />
+    <axis xyz="0.640206045739845 0 0.768203240684489" />
   </joint>
   <link name="LL2_coxa">
     <inertial>
-      <origin xyz="0.0127223107624808 0.0169176334399643 -0.0226841712591478" rpy="0 0 0" />
-      <mass value="0.011831113051677" />
-      <inertia ixx="1.56088112402009E-06" ixy="-2.81601853556498E-08" ixz="2.19396104805269E-08" iyy="1.03946591481982E-06" iyz="-2.12255249861136E-08" izz="1.4607575411285E-06" />
+      <origin xyz="0.0127223100660754 0.0169176353715654 -0.0226841740829874" rpy="0 0 0" />
+      <mass value="0.0118311161508981" />
+      <inertia ixx="1.56088144680102E-06" ixy="-2.81600783319572E-08" ixz="2.19394756026617E-08" iyy="1.03946603017998E-06" iyz="-2.12253461630087E-08" izz="1.46075766684656E-06" />
     </inertial>
     <visual>
@@ -471,5 +471,5 @@
   </link>
   <joint name="joint6_coxa" type="continuous">
-    <origin xyz="0.0870706319702601 0.0399393134553608 0.00464999999999998" rpy="1.5707963267949 0 0.840128894013488" />
+    <origin xyz="0.0614346512851298 0.0483293208043272 0.00180390069504796" rpy="1.5707963267949 0 0.799360343333685" />
     <parent link="base_link" />
     <child link="LL2_coxa" />
@@ -478,7 +478,7 @@
   <link name="LL2_fumer">
     <inertial>
-      <origin xyz="-0.0264233888332989 4.16333634234434E-17 0.0725596957982222" rpy="0 0 0" />
+      <origin xyz="-0.0264233888332986 0 0.0120596957982234" rpy="0 0 0" />
       <mass value="0.00732061922605988" />
-      <inertia ixx="1.66034801156123E-06" ixy="-9.52912065661088E-22" ixz="-1.49987503139381E-09" iyy="3.33489508651991E-06" iyz="-3.12570873968475E-22" izz="1.85153973126671E-06" />
+      <inertia ixx="1.66034801156124E-06" ixy="1.05879118406788E-22" ixz="-1.49987503139611E-09" iyy="3.33489508651991E-06" iyz="5.09543257332665E-22" izz="1.85153973126671E-06" />
     </inertial>
     <visual>
@@ -499,5 +499,5 @@
   </link>
   <joint name="joint6_fumer" type="continuous">
-    <origin xyz="0.0608557453435872 0.0221 0.026703525210662" rpy="-2.72035311532009 -0.616222550074482 2.48212725475599" />
+    <origin xyz="0.0204800515080549 0.0220999999999997 -0.0183525881070598" rpy="-2.71143718885399 -0.610479400867026 2.46663802210369" />
     <parent link="LL2_coxa" />
     <child link="LL2_fumer" />
@@ -506,7 +506,7 @@
   <link name="LL2_tibia">
     <inertial>
-      <origin xyz="-0.01480952139402 -0.013098396107006 -0.0165422174946064" rpy="0 0 0" />
-      <mass value="0.013123891605465" />
-      <inertia ixx="4.36428688191597E-06" ixy="-2.1723438599018E-07" ixz="-8.58851441227647E-08" iyy="7.89056082804284E-07" iyz="2.68586343447735E-07" izz="4.28337682704655E-06" />
+      <origin xyz="-0.00780217032358205 -0.01309839267037 -0.00872256326972962" rpy="0 0 0" />
+      <mass value="0.0131238944675766" />
+      <inertia ixx="4.36428717131208E-06" ixy="-2.17234269804496E-07" ixz="-8.58852825162038E-08" iyy="7.89056187070732E-07" iyz="2.6858651802412E-07" izz="4.28337690198118E-06" />
     </inertial>
     <visual>
@@ -527,14 +527,14 @@
   </link>
   <joint name="joint6_tibia" type="continuous">
-    <origin xyz="-0.0549999999999999 0 0.0500000000000001" rpy="3.14159265358979 0.730667432781409 2.60353309806751" />
+    <origin xyz="-0.055 0 0" rpy="3.14159265358979 0.730667432781409 2.63033642671627" />
     <parent link="LL2_fumer" />
     <child link="LL2_tibia" />
-    <axis xyz="0.667366840256722 0 0.744729145747471" />
+    <axis xyz="0.667366840256722 0 0.744729145747472" />
   </joint>
   <link name="LL3_coxa">
     <inertial>
-      <origin xyz="0.0139602506872404 0.0172339889705058 -0.0204671642059132" rpy="0 0 0" />
-      <mass value="0.011831113051677" />
-      <inertia ixx="1.46157119792145E-06" ixy="-2.17239801391936E-08" ixz="2.37095554539396E-08" iyy="1.03946591481982E-06" iyz="-2.7777459121755E-08" izz="1.56006746722729E-06" />
+      <origin xyz="0.0139602506469437 0.0172339889077581 -0.0204671641770284" rpy="0 0 0" />
+      <mass value="0.0118311133553872" />
+      <inertia ixx="1.46157125552418E-06" ixy="-2.17239736681064E-08" ixz="2.37095607651922E-08" iyy="1.0394659305145E-06" iyz="-2.77774755690175E-08" izz="1.56006751193327E-06" />
     </inertial>
     <visual>
@@ -555,5 +555,5 @@
   </link>
   <joint name="joint7_coxa" type="continuous">
-    <origin xyz="0.0265706319702602 0.0399393134553611 0.00464999999999998" rpy="1.5707963267949 0 0.712846787592376" />
+    <origin xyz="0.00143606445544368 0.0405563176240433 0.0018039006950479" rpy="1.5707963267949 0 0.762566282617874" />
     <parent link="base_link" />
     <child link="LL3_coxa" />
@@ -562,7 +562,7 @@
   <link name="LL3_fumer">
     <inertial>
-      <origin xyz="-0.0264233888332988 1.66533453693773E-16 0.125559695798222" rpy="0 0 0" />
-      <mass value="0.00732061922605986" />
-      <inertia ixx="1.66034801156123E-06" ixy="4.76456032830544E-22" ixz="-1.49987503139544E-09" iyy="3.3348950865199E-06" iyz="1.16058502206239E-22" izz="1.85153973126671E-06" />
+      <origin xyz="-0.0264233888332985 -1.38777878078145E-17 0.00455969579822281" rpy="0 0 0" />
+      <mass value="0.00732061922605988" />
+      <inertia ixx="1.66034801156124E-06" ixy="-6.88214269644119E-22" ixz="-1.49987503139482E-09" iyy="3.3348950865199E-06" iyz="-2.64697796016969E-22" izz="1.85153973126671E-06" />
     </inertial>
     <visual>
@@ -583,5 +583,5 @@
   </link>
   <joint name="joint7_fumer" type="continuous">
-    <origin xyz="0.10952160956792 0.0221 0.0583289553965433" rpy="-2.61722554755421 -0.71438242643614 2.41835522432309" />
+    <origin xyz="0.0179847256047489 0.0221 -0.0208038372643574" rpy="-2.66841470881931 -0.745546268941601 2.49508842776342" />
     <parent link="LL3_coxa" />
     <child link="LL3_fumer" />
@@ -590,7 +590,7 @@
   <link name="LL3_tibia">
     <inertial>
-      <origin xyz="-0.094631241235736 -0.00999543048455966 -0.0821821673541989" rpy="0 0 0" />
-      <mass value="0.021123795973342" />
-      <inertia ixx="4.99508664772741E-06" ixy="-1.3939361777078E-07" ixz="-2.6733864336624E-07" iyy="1.32635282258011E-06" iyz="1.78140065284283E-07" izz="5.01286567758949E-06" />
+      <origin xyz="-0.00309435726524095 -0.00999543050929356 -0.00304937467236494" rpy="0 0 0" />
+      <mass value="0.0211237959439876" />
+      <inertia ixx="4.9950866400634E-06" ixy="-1.39393620012794E-07" ixz="-2.67338640754455E-07" iyy="1.32635281980292E-06" iyz="1.78140060908311E-07" izz="5.01286567504397E-06" />
     </inertial>
     <visual>
@@ -611,5 +611,5 @@
   </link>
   <joint name="joint7_tibia" type="continuous">
-    <origin xyz="-0.0549999999999999 0 0" rpy="3.14159265358979 0.857949539202522 2.63388766827357" />
+    <origin xyz="-0.0549999999999996 0 0" rpy="-3.14159265358979 0.857949539202521 2.68310369735863" />
     <parent link="LL3_fumer" />
     <child link="LL3_tibia" />
@@ -618,7 +618,7 @@
   <link name="LL4_coxa">
     <inertial>
-      <origin xyz="0.000589847633677063 0.017230005966643 -0.0246801710229706" rpy="0 0 0" />
-      <mass value="0.0118214531865818" />
-      <inertia ixx="1.53674766199004E-06" ixy="3.56106840430809E-08" ixz="-4.78840740951851E-08" iyy="1.03828147386784E-06" iyz="-3.33600105752004E-09" izz="1.48303577587997E-06" />
+      <origin xyz="0.000589847914708751 0.0172300062160811 -0.0246801710520806" rpy="0 0 0" />
+      <mass value="0.0118214537178174" />
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