Commit message: circle gait added _ spider_desc initial pose error rectfied _ meshes readded

File: spider_description/urdf/spider_description.xacro (robot description, xacro)
@@ -8,7 +8,7 @@
   <link name="base_link">
     <inertial>
-      <origin xyz="0.0419124697856288 0.00194512919498489 0.0129912705123136" rpy="0 0 0" />
+      <origin xyz="0.0419124697856288 0.0129912705123136 -0.00194512919498489" rpy="0 0 0" />
       <mass value="0.206593361987693" />
-      <inertia ixx="0.000100835459421752" ixy="-6.85143109069959E-05" ixz="3.31903264428765E-07" iyy="0.000612159753876248" iyz="7.47632670675686E-08" izz="0.000699628428109392" />
+      <inertia ixx="0.000100835459421752" ixy="3.3190326442876E-07" ixz="6.85143109069958E-05" iyy="0.000699628428109392" iyz="-7.47632670675628E-08" izz="0.000612159753876248" />
     </inertial>
     <visual>
@@ -30,7 +30,7 @@
   <link name="RL1_coxa">
     <inertial>
-      <origin xyz="-0.00349164005789518 0.0172300074490141 0.0244390510670151" rpy="0 0 0" />
-      <mass value="0.0118214567647082" />
-      <inertia ixx="1.54720121311925E-06" ixy="-3.57556897862798E-08" ixz="-4.02761529137734E-08" iyy="1.03828172792338E-06" iyz="-8.80256909637123E-10" izz="1.47258341600743E-06" />
+      <origin xyz="-0.00349163991648843 0.0172300072694273 0.024439051068252" rpy="0 0 0" />
+      <mass value="0.0118214563639757" />
+      <inertia ixx="1.54720113656629E-06" ixy="-3.57556957341545E-08" ixz="-4.0276165283765E-08" iyy="1.03828170219183E-06" iyz="-8.80235914490984E-10" izz="1.47258336300693E-06" />
     </inertial>
     <visual>
@@ -51,15 +51,14 @@
   </link>
   <joint name="joint1_coxa" type="continuous">
-    <origin xyz="0.14302 -0.028828 0.0018039" rpy="1.5708 0 0.60122" />
+    <origin xyz="0.143023923046985 -0.028827601978856 0.00180390069504784" rpy="1.5707963267949 0 0.456646809528589" />
     <parent link="base_link" />
     <child link="RL1_coxa" />
     <axis xyz="0 1 0" />
-    <limit effort="20.0" velocity="1.0" />
   </joint>
   <link name="RL1_fumer">
     <inertial>
-      <origin xyz="-0.0264233888332986 -1.38777878078145E-17 -0.00234030420177818" rpy="0 0 0" />
-      <mass value="0.00732061922605989" />
-      <inertia ixx="1.66034801156124E-06" ixy="-5.29395592033938E-22" ixz="-1.49987503139451E-09" iyy="3.33489508651992E-06" iyz="-2.11758236813575E-22" izz="1.85153973126671E-06" />
+      <origin xyz="-0.0264233888332986 6.93889390390723E-18 -0.00234030420177805" rpy="0 0 0" />
+      <mass value="0.00732061922605988" />
+      <inertia ixx="1.66034801156124E-06" ixy="1.00585162486448E-21" ixz="-1.49987503139991E-09" iyy="3.33489508651991E-06" iyz="1.04555629426703E-21" izz="1.85153973126671E-06" />
     </inertial>
     <visual>
@@ -80,15 +79,14 @@
   </link>
   <joint name="joint1_fumer" type="continuous">
-    <origin xyz="-0.0059198 0.0221 0.026855" rpy="-2.0354 1.0696 1.1567" />
+    <origin xyz="-0.00591979008225604 0.0221000000000001 0.026855280400361" rpy="-2.03537963970565 1.06963032129347 1.15667679281028" />
     <parent link="RL1_coxa" />
     <child link="RL1_fumer" />
     <axis xyz="0 0 1" />
-    <limit effort="20.0" velocity="1.0" />
   </joint>
   <link name="RL1_tibia">
     <inertial>
-      <origin xyz="0.0026015472226265 -0.0130975375884837 0.000727426107816176" rpy="0 0 0" />
-      <mass value="0.0131238915537926" />
-      <inertia ixx="4.22996621810264E-06" ixy="1.19149401954703E-07" ixz="-1.17548940136716E-08" iyy="7.82194138869205E-07" iyz="-2.83284563170215E-07" izz="4.42455940433514E-06" />
+      <origin xyz="0.00260154719028149 -0.013097537565338 0.000727426101389261" rpy="0 0 0" />
+      <mass value="0.0131238915671885" />
+      <inertia ixx="4.22996621859555E-06" ixy="1.19149405996142E-07" ixz="-1.17548949137053E-08" iyy="7.82194141970863E-07" iyz="-2.83284562385563E-07" izz="4.4245594105805E-06" />
     </inertial>
     <visual>
@@ -109,15 +107,14 @@
   </link>
   <joint name="joint1_tibia" type="continuous">
-    <origin xyz="-0.055 0 0" rpy="3.14159265358979 1.35383304701328 0.45541675484875" />
+    <origin xyz="-0.055 0 0" rpy="3.14159265358979 1.35383304701328 0.455416754848752" />
     <parent link="RL1_fumer" />
     <child link="RL1_tibia" />
-    <axis xyz="0.976555650922224 0 0.21526509390022" />
-    <limit effort="20.0" velocity="1.0" />
+    <axis xyz="0.976555650922224 0 0.215265093900221" />
   </joint>
   <link name="RL2_coxa">
     <inertial>
-      <origin xyz="-0.00137410436525083 0.0172300079511928 0.0246489469646006" rpy="0 0 0" />
-      <mass value="0.0118214569541968" />
-      <inertia ixx="1.53973642077788E-06" ixy="-3.56985158373652E-08" ixz="-4.60808282191804E-08" iyy="1.0382816314569E-06" iyz="2.20230674733217E-09" izz="1.48004767988558E-06" />
+      <origin xyz="-0.00137410359807341 0.0172300072704422 0.0246489473554496" rpy="0 0 0" />
+      <mass value="0.0118214563661804" />
+      <inertia ixx="1.53973680405956E-06" ixy="-3.56986723887601E-08" ixz="-4.6080637183373E-08" iyy="1.0382817023383E-06" iyz="2.2021308274049E-09" izz="1.4800476962292E-06" />
     </inertial>
     <visual>
@@ -138,15 +135,14 @@
   </link>
   <joint name="joint2_coxa" type="continuous">
-    <origin xyz="0.083025 -0.036601 0.0018039" rpy="1.5708 0 0" />
+    <origin xyz="0.0830253362173002 -0.0366006051591393 0.00180390069504788" rpy="1.5707963267949 0 0.371215936961481" />
     <parent link="base_link" />
     <child link="RL2_coxa" />
     <axis xyz="0 1 0" />
-    <limit effort="20.0" velocity="1.0" />
   </joint>
   <link name="RL2_fumer">
     <inertial>
-      <origin xyz="-0.0264233888332986 1.38777878078145E-17 -0.00234030420177736" rpy="0 0 0" />
+      <origin xyz="-0.0264233888332985 0 -0.00234030420177726" rpy="0 0 0" />
       <mass value="0.00732061922605988" />
-      <inertia ixx="1.66034801156124E-06" ixy="5.29395592033938E-23" ixz="-1.49987503139717E-09" iyy="3.33489508651991E-06" iyz="1.05879118406788E-22" izz="1.85153973126671E-06" />
+      <inertia ixx="1.66034801156124E-06" ixy="3.70576914423756E-22" ixz="-1.49987503139454E-09" iyy="3.33489508651991E-06" iyz="-2.5146290621612E-22" izz="1.85153973126671E-06" />
     </inertial>
     <visual>
@@ -167,15 +163,14 @@
   </link>
   <joint name="joint2_fumer" type="continuous">
-    <origin xyz="-0.00358516044020271 0.0220999999999999 0.027265300743216" rpy="-1.96635013509526 1.22564253387824 1.19639468178544" />
+    <origin xyz="-0.00358516044020296 0.0220999999999999 0.0272653007432159" rpy="-1.84005724604345 1.0586197588623 1.33473036772911" />
     <parent link="RL2_coxa" />
     <child link="RL2_fumer" />
     <axis xyz="0 0 1" />
-    <limit effort="20.0" velocity="1.0" />
   </joint>
   <link name="RL2_tibia">
     <inertial>
-      <origin xyz="0.00373414548593776 -0.0130839558065926 0.00111120131468931" rpy="0 0 0" />
-      <mass value="0.0131238945709346" />
-      <inertia ixx="4.23019156808467E-06" ixy="7.84255900620934E-08" ixz="1.01964592236264E-09" iyy="7.65338600134478E-07" iyz="-1.63714042120736E-07" izz="4.4411901162674E-06" />
+      <origin xyz="0.00373414734956586 -0.0130839594099826 0.00111120240408577" rpy="0 0 0" />
+      <mass value="0.0131238915536145" />
+      <inertia ixx="4.23019149640981E-06" ixy="7.84253770640042E-08" ixz="1.01978479704144E-09" iyy="7.6533847696787E-07" iyz="-1.63714108486507E-07" izz="4.44118979210614E-06" />
     </inertial>
     <visual>
@@ -196,15 +191,14 @@
   </link>
   <joint name="joint2_tibia" type="continuous">
-    <origin xyz="-0.055 0 0" rpy="-3.1416 1.4401 0.32035" />
+    <origin xyz="-0.055 0 0" rpy="-3.14159265358979 1.4400547052635 0.436973540292822" />
     <parent link="RL2_fumer" />
     <child link="RL2_tibia" />
-    <axis xyz="0.99147 0 0.13037" />
-    <limit effort="20.0" velocity="1.0" />
+    <axis xyz="0.991465481571485 0 0.130369470552824" />
   </joint>
   <link name="RL3_coxa">
     <inertial>
-      <origin xyz="0.00349357804156721 0.0172300087939702 0.0244387737682328" rpy="0 0 0" />
-      <mass value="0.0118214592735859" />
-      <inertia ixx="1.51968707139066E-06" ixy="-3.45707433343636E-08" ixz="-5.4020292631234E-08" iyy="1.0382817957142E-06" iyz="9.17029253519079E-09" izz="1.50009780239266E-06" />
+      <origin xyz="0.00349358017075859 0.01723000702548 0.0244387737829021" rpy="0 0 0" />
+      <mass value="0.0118214556819711" />
+      <inertia ixx="1.51968692035686E-06" ixy="-3.45709549158988E-08" ixz="-5.40202304528258E-08" iyy="1.03828165876939E-06" iyz="9.17031077224167E-09" izz="1.50009735512406E-06" />
     </inertial>
     <visual>
@@ -225,15 +219,14 @@
   </link>
   <joint name="joint3_coxa" type="continuous">
-    <origin xyz="0.0230267493876147 -0.0443736083394228 0.00180390069504786" rpy="1.5707963267949 0 -0.472149585715113" />
+    <origin xyz="0.0230267493876147 -0.0443736083394228 0.00180390069504786" rpy="1.5707963267949 0 0.115999004572643" />
     <parent link="base_link" />
     <child link="RL3_coxa" />
     <axis xyz="0 1 0" />
-    <limit effort="20.0" velocity="1.0" />
   </joint>
   <link name="RL3_fumer">
     <inertial>
-      <origin xyz="-0.0264233888332986 -1.38777878078145E-17 -0.00234030420177761" rpy="0 0 0" />
-      <mass value="0.00732061922605987" />
-      <inertia ixx="1.66034801156124E-06" ixy="-1.16467030247466E-21" ixz="-1.49987503139679E-09" iyy="3.33489508651991E-06" iyz="-8.99972506457694E-22" izz="1.85153973126671E-06" />
+      <origin xyz="-0.0190060888231168 -0.0093450118645113 -0.00493699671842929" rpy="0 0 0" />
+      <mass value="0.00732061922605988" />
+      <inertia ixx="1.66034801156124E-06" ixy="-8.470329472543E-22" ixz="-1.4998750313965E-09" iyy="3.33489508651991E-06" iyz="-6.61744490042422E-23" izz="1.85153973126671E-06" />
     </inertial>
     <visual>
@@ -254,15 +247,14 @@
   </link>
   <joint name="joint3_fumer" type="continuous">
-    <origin xyz="0.00183942151113823 0.0220999999999999 0.0274384133743986" rpy="-1.48461478428462 0.680765280133814 1.62511913782005" />
+    <origin xyz="-0.000624989213601535 0.0103198993706474 0.0294985850073072" rpy="-1.43474773528477 1.05506840370706 1.68932703577979" />
     <parent link="RL3_coxa" />
     <child link="RL3_fumer" />
     <axis xyz="0 0 1" />
-    <limit effort="20.0" velocity="1.0" />
   </joint>
   <link name="RL3_tibia">
     <inertial>
-      <origin xyz="0.00272348248477123 -0.0130894484904979 0.000302596670154601" rpy="0 0 0" />
-      <mass value="0.0131238945459342" />
-      <inertia ixx="4.23878067567191E-06" ixy="4.20084297779206E-08" ixz="4.1875712377848E-08" iyy="7.69154583662019E-07" iyz="-2.12494139960766E-07" izz="4.42878502193697E-06" />
+      <origin xyz="0.00531436167769063 -0.0130894520266102 0.000128909648472023" rpy="0 0 0" />
+      <mass value="0.013123891554142" />
+      <inertia ixx="4.23878064857726E-06" ixy="4.20082179122996E-08" ixz="4.18757972044376E-08" iyy="7.69154455506806E-07" iyz="-2.12494162555612E-07" izz="4.42878466326275E-06" />
     </inertial>
     <visual>
@@ -283,15 +275,14 @@
   </link>
   <joint name="joint3_tibia" type="continuous">
-    <origin xyz="-0.055 0 0" rpy="0 1.50385829483433 -2.56000504688249" />
+    <origin xyz="-0.0475826999898183 -0.0093450118645113 0" rpy="0 1.50385829483433 -2.6917648290032" />
     <parent link="RL3_fumer" />
     <child link="RL3_tibia" />
-    <axis xyz="0.997760486341758 0 -0.0668880549504797" />
-    <limit effort="20.0" velocity="1.0" />
+    <axis xyz="0.997760486341758 0 -0.0668880549504796" />
   </joint>
   <link name="RL4_coxa">
     <inertial>
-      <origin xyz="0.000221645762317584 0.017233990044243 0.0247738647215934" rpy="0 0 0" />
-      <mass value="0.0118311173645293" />
-      <inertia ixx="1.51589418009088E-06" ixy="3.36931862404341E-08" ixz="5.44220173389888E-08" iyy="1.03946613397378E-06" iyz="1.04055920493148E-08" izz="1.50574537269555E-06" />
+      <origin xyz="0.000221643431956145 0.0172339886263365 0.024773862822896" rpy="0 0 0" />
+      <mass value="0.0118311142541974" />
+      <inertia ixx="1.51589405750511E-06" ixy="3.36933854050161E-08" ixz="5.44221416465647E-08" iyy="1.03946598429508E-06" iyz="1.04056213225627E-08" izz="1.50574501931213E-06" />
     </inertial>
     <visual>
@@ -312,15 +303,14 @@
   </link>
   <joint name="joint4_coxa" type="continuous">
-    <origin xyz="-0.036972 -0.052147 0.0018039" rpy="1.5708 0 0" />
+    <origin xyz="-0.0369718374420689 -0.0521466115197065 0.00180390069504695" rpy="1.5707963267949 0 0.279272825129561" />
     <parent link="base_link" />
     <child link="RL4_coxa" />
     <axis xyz="0 1 0" />
-    <limit effort="20.0" velocity="1.0" />
   </joint>
   <link name="RL4_fumer">
     <inertial>
-      <origin xyz="-0.0264233888332986 -1.38777878078145E-17 0.00455969579822268" rpy="0 0 0" />
-      <mass value="0.00732061922605988" />
-      <inertia ixx="1.66034801156124E-06" ixy="5.29395592033938E-22" ixz="-1.49987503139543E-09" iyy="3.33489508651991E-06" iyz="3.30872245021211E-22" izz="1.85153973126671E-06" />
+      <origin xyz="-0.0264233888332986 -1.38777878078145E-17 0.00455969579822089" rpy="0 0 0" />
+      <mass value="0.00732061922605989" />
+      <inertia ixx="1.66034801156124E-06" ixy="-1.11173074327127E-21" ixz="-1.49987503139615E-09" iyy="3.33489508651992E-06" iyz="-8.73502726855997E-22" izz="1.85153973126671E-06" />
     </inertial>
     <visual>
@@ -341,15 +331,14 @@
   </link>
   <joint name="joint4_fumer" type="continuous">
-    <origin xyz="-0.0028905 0.0221 0.027348" rpy="1.4151 0.82627 1.4558" />
+    <origin xyz="-0.00289047043580869 0.0221000000000014 0.0273476723078892" rpy="1.34757833958992 1.0760490052699 1.37361152936902" />
     <parent link="RL4_coxa" />
     <child link="RL4_fumer" />
     <axis xyz="0 0 1" />
-    <limit effort="20.0" velocity="1.0" />
   </joint>
   <link name="RL4_tibia">
     <inertial>
-      <origin xyz="0.00461943235034938 -0.0124119057494399 -0.00371988244958756" rpy="0 0 0" />
-      <mass value="0.0131238915832408" />
-      <inertia ixx="4.23942335671897E-06" ixy="1.02033757545884E-07" ixz="-4.08466849980063E-09" iyy="1.36774622760594E-06" iyz="-1.36758688235976E-06" izz="3.82955020041708E-06" />
+      <origin xyz="0.0046194323285307 -0.0124119057556658 -0.00371988245181533" rpy="0 0 0" />
+      <mass value="0.0131238915753325" />
+      <inertia ixx="4.23942335586469E-06" ixy="1.02033759025192E-07" ixz="-4.08466826831512E-09" iyy="1.36774622353105E-06" iyz="-1.36758688276913E-06" izz="3.82955019670378E-06" />
     </inertial>
     <visual>
@@ -370,15 +359,14 @@
   </link>
   <joint name="joint4_tibia" type="continuous">
-    <origin xyz="-0.0550000000000007 0 0" rpy="0 -1.4654938088774 -0.738464203109028" />
+    <origin xyz="-0.0550000000000001 0 0" rpy="0 -1.4654938088774 -0.809353512947539" />
     <parent link="RL4_fumer" />
     <child link="RL4_tibia" />
     <axis xyz="0.994460811195995 0 0.105108015847522" />
-    <limit effort="20.0" velocity="1.0" />
   </joint>
   <link name="LL1_coxa">
     <inertial>
-      <origin xyz="0.0170998829456735 0.0172339868446963 -0.0179272815287505" rpy="0 0 0" />
-      <mass value="0.0118311175968466" />
-      <inertia ixx="1.45657032662236E-06" ixy="-1.69225127081701E-08" ixz="6.6690604598061E-09" iyy="1.0394662195964E-06" iyz="-3.09379598799848E-08" izz="1.56506993041627E-06" />
+      <origin xyz="0.0170998824043466 0.0172339901017211 -0.017927284271033" rpy="0 0 0" />
+      <mass value="0.0118311172441887" />
+      <inertia ixx="1.45657003099262E-06" ixy="-1.69225042702206E-08" ixz="6.66881674443564E-09" iyy="1.03946612492756E-06" iyz="-3.09376104608946E-08" izz="1.5650694795515E-06" />
     </inertial>
     <visual>
@@ -399,15 +387,14 @@
   </link>
   <joint name="joint5_coxa" type="continuous">
-    <origin xyz="0.12143 0.056102 0.0018039" rpy="1.5708 0 -0.12925" />
+    <origin xyz="0.121433238114814 0.0561023239846096 0.00180390069504789" rpy="1.5707963267949 0 0.779171496523206" />
     <parent link="base_link" />
     <child link="LL1_coxa" />
     <axis xyz="0 1 0" />
-    <limit effort="20.0" velocity="1.0" />
   </joint>
   <link name="LL1_fumer">
     <inertial>
-      <origin xyz="-0.0264233888332986 -1.38777878078145E-17 0.00455969579822259" rpy="0 0 0" />
+      <origin xyz="-0.0264233888332985 0 0.00455969579822237" rpy="0 0 0" />
       <mass value="0.00732061922605988" />
-      <inertia ixx="1.66034801156124E-06" ixy="-9.79381845262785E-22" ixz="-1.49987503139472E-09" iyy="3.33489508651991E-06" iyz="-1.6940658945086E-21" izz="1.85153973126671E-06" />
+      <inertia ixx="1.66034801156124E-06" ixy="5.29395592033938E-22" ixz="-1.49987503139699E-09" iyy="3.33489508651991E-06" iyz="-4.2351647362715E-22" izz="1.85153973126671E-06" />
     </inertial>
     <visual>
@@ -428,15 +415,14 @@
   </link>
   <joint name="joint5_fumer" type="continuous">
-    <origin xyz="0.0211255891188235 0.0220999999999999 -0.0176056662578459" rpy="-2.67256230035857 -0.533155379057018 2.35767887359705" />
+    <origin xyz="0.0211255891188228 0.0221 -0.0176056662578466" rpy="-2.73801909944616 -0.582101669425183 2.48122445090949" />
     <parent link="LL1_coxa" />
     <child link="LL1_fumer" />
     <axis xyz="0 0 1" />
-    <limit effort="20.0" velocity="1.0" />
   </joint>
   <link name="LL1_tibia">
     <inertial>
-      <origin xyz="-0.00279894253481278 -0.0130976425422804 -0.0031384336970829" rpy="0 0 0" />
-      <mass value="0.0131238915475162" />
-      <inertia ixx="4.36602524922464E-06" ixy="-2.59110660060209E-07" ixz="-7.85274834003549E-08" iyy="7.97432594738258E-07" iyz="2.87128223672932E-07" izz="4.27326190737941E-06" />
+      <origin xyz="-0.00279894329842953 -0.0130976389443435 -0.00313843570289792" rpy="0 0 0" />
+      <mass value="0.0131238945399001" />
+      <inertia ixx="4.36602557276728E-06" ixy="-2.59110541265302E-07" ixz="-7.85276269962679E-08" iyy="7.97432719732035E-07" iyz="2.87128419374741E-07" izz="4.27326198471528E-06" />
     </inertial>
     <visual>
@@ -457,15 +443,14 @@
   </link>
   <joint name="joint5_tibia" type="continuous">
-    <origin xyz="-0.055 0 0" rpy="-3.14159265358979 0.694766453403042 2.4879765741821" />
+    <origin xyz="-0.0549999999999999 0 0" rpy="-3.14159265358979 0.69476645340304 2.60363290009658" />
     <parent link="LL1_fumer" />
     <child link="LL1_tibia" />
-    <axis xyz="0.640206045739847 0 0.768203240684488" />
-    <limit effort="20.0" velocity="1.0" />
+    <axis xyz="0.640206045739845 0 0.768203240684489" />
   </joint>
   <link name="LL2_coxa">
     <inertial>
-      <origin xyz="0.0127223136312809 0.0169176380368381 -0.0226841698345239" rpy="0 0 0" />
-      <mass value="0.0118311153864136" />
-      <inertia ixx="1.56088145996956E-06" ixy="-2.81605475151796E-08" ixz="2.19397573465521E-08" iyy="1.03946620496031E-06" iyz="-2.12254323475495E-08" izz="1.46075806401663E-06" />
+      <origin xyz="0.0127223100660754 0.0169176353715654 -0.0226841740829874" rpy="0 0 0" />
+      <mass value="0.0118311161508981" />
+      <inertia ixx="1.56088144680102E-06" ixy="-2.81600783319572E-08" ixz="2.19394756026617E-08" iyy="1.03946603017998E-06" iyz="-2.12253461630087E-08" izz="1.46075766684656E-06" />
     </inertial>
     <visual>
@@ -486,15 +471,14 @@
   </link>
   <joint name="joint6_coxa" type="continuous">
-    <origin xyz="0.061435 0.048329 0.0018039" rpy="1.5708 0 0" />
+    <origin xyz="0.0614346512851298 0.0483293208043272 0.00180390069504796" rpy="1.5707963267949 0 0.799360343333685" />
     <parent link="base_link" />
     <child link="LL2_coxa" />
     <axis xyz="0 1 0" />
-    <limit effort="20.0" velocity="1.0" />
   </joint>
   <link name="LL2_fumer">
     <inertial>
-      <origin xyz="-0.0264233888332986 -1.38777878078145E-17 0.0120596957982223" rpy="0 0 0" />
+      <origin xyz="-0.0264233888332986 0 0.0120596957982234" rpy="0 0 0" />
       <mass value="0.00732061922605988" />
-      <inertia ixx="1.66034801156124E-06" ixy="-6.68361934942846E-22" ixz="-1.49987503139737E-09" iyy="3.33489508651991E-06" iyz="4.76456032830544E-22" izz="1.85153973126671E-06" />
+      <inertia ixx="1.66034801156124E-06" ixy="1.05879118406788E-22" ixz="-1.49987503139611E-09" iyy="3.33489508651991E-06" iyz="5.09543257332665E-22" izz="1.85153973126671E-06" />
     </inertial>
     <visual>
@@ -515,15 +499,14 @@
   </link>
   <joint name="joint6_fumer" type="continuous">
-    <origin xyz="0.0204800515080558 0.0220999999999999 -0.0183525881070601" rpy="-3.06812253072566 -0.727643744163724 3.03137911431499" />
+    <origin xyz="0.0204800515080549 0.0220999999999997 -0.0183525881070598" rpy="-2.71143718885399 -0.610479400867026 2.46663802210369" />
     <parent link="LL2_coxa" />
     <child link="LL2_fumer" />
     <axis xyz="0 0 1" />
-    <limit effort="20.0" velocity="1.0" />
   </joint>
   <link name="LL2_tibia">
     <inertial>
-      <origin xyz="-0.00780216947933945 -0.0130983962022635 -0.00872256136528804" rpy="0 0 0" />
-      <mass value="0.0131238915503292" />
-      <inertia ixx="4.36428686800826E-06" ixy="-2.172343973603E-07" ixz="-8.58851317959739E-08" iyy="7.89056070109124E-07" iyz="2.68586330967299E-07" izz="4.28337681328811E-06" />
+      <origin xyz="-0.00780217032358205 -0.01309839267037 -0.00872256326972962" rpy="0 0 0" />
+      <mass value="0.0131238944675766" />
+      <inertia ixx="4.36428717131208E-06" ixy="-2.17234269804496E-07" ixz="-8.58852825162038E-08" iyy="7.89056187070732E-07" iyz="2.6858651802412E-07" izz="4.28337690198118E-06" />
     </inertial>
     <visual>
@@ -544,15 +527,14 @@
   </link>
   <joint name="joint6_tibia" type="continuous">
-    <origin xyz="-0.055 0 0" rpy="3.14159265358979 0.730667432781408 3.05936528141118" />
+    <origin xyz="-0.055 0 0" rpy="3.14159265358979 0.730667432781409 2.63033642671627" />
     <parent link="LL2_fumer" />
     <child link="LL2_tibia" />
-    <axis xyz="0.667366840256722 0 0.744729145747471" />
-    <limit effort="20.0" velocity="1.0" />
+    <axis xyz="0.667366840256722 0 0.744729145747472" />
   </joint>
   <link name="LL3_coxa">
     <inertial>
-      <origin xyz="0.0139602511615753 0.0172339841699638 -0.0204671653605546" rpy="0 0 0" />
-      <mass value="0.011831115338393" />
-      <inertia ixx="1.46157171906711E-06" ixy="-2.17238956764402E-08" ixz="2.37096972238414E-08" iyy="1.03946620191304E-06" iyz="-2.7777820329616E-08" izz="1.56006778830444E-06" />
+      <origin xyz="0.0139602506469437 0.0172339889077581 -0.0204671641770284" rpy="0 0 0" />
+      <mass value="0.0118311133553872" />
+      <inertia ixx="1.46157125552418E-06" ixy="-2.17239736681064E-08" ixz="2.37095607651922E-08" iyy="1.0394659305145E-06" iyz="-2.77774755690175E-08" izz="1.56006751193327E-06" />
     </inertial>
     <visual>
@@ -573,15 +555,14 @@
   </link>
   <joint name="joint7_coxa" type="continuous">
-    <origin xyz="0.00143606445544368 0.0405563176240433 0.0018039006950479" rpy="1.5707963267949 0 0" />
+    <origin xyz="0.00143606445544368 0.0405563176240433 0.0018039006950479" rpy="1.5707963267949 0 0.762566282617874" />
     <parent link="base_link" />
     <child link="LL3_coxa" />
     <axis xyz="0 1 0" />
-    <limit effort="20.0" velocity="1.0" />
   </joint>
   <link name="LL3_fumer">
     <inertial>
-      <origin xyz="-0.0264233888332986 -6.93889390390723E-18 0.00455969579822243" rpy="0 0 0" />
+      <origin xyz="-0.0264233888332985 -1.38777878078145E-17 0.00455969579822281" rpy="0 0 0" />
       <mass value="0.00732061922605988" />
-      <inertia ixx="1.66034801156124E-06" ixy="1.58818677610181E-22" ixz="-1.49987503139568E-09" iyy="3.33489508651991E-06" iyz="5.82335151237331E-22" izz="1.85153973126671E-06" />
+      <inertia ixx="1.66034801156124E-06" ixy="-6.88214269644119E-22" ixz="-1.49987503139482E-09" iyy="3.3348950865199E-06" iyz="-2.64697796016969E-22" izz="1.85153973126671E-06" />
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