Commit message: added lidar and camera

File: spider_description/urdf/spider_description.xacro (robot description, xacro)
@@ -1,3 +1,7 @@
-<robot name="spider_description">
+<?xml version="1.0"?>
+<robot xmlns:xacro="http://www.ros.org/wiki/xacro" name="spider_description">
+  <xacro:include filename="$(find spider_description)/urdf/lidar.gazebo" />
+  <xacro:include filename="$(find spider_description)/urdf/realsense2_camera.xacro" />
+  <!-- <xacro:include filename="camera.xacro" /> -->
   <link name="dummy_base" />
   <joint name="dummy_base_to_base_link" type="fixed">
@@ -10,19 +14,19 @@
       <origin xyz="0.0513553543804905 -0.00355010292388771 0.0158371951293718" rpy="0 0 0" />
       <mass value="0.206587820695411" />
-      <inertia ixx="9.18101041743378E-05" ixy="-1.1096915717602E-06" ixz="-2.07334737671996E-08" iyy="0.000621158029436724" iyz="3.17880975410803E-08" izz="0.000699601373790156" />
-    </inertial>
-    <visual>
-      <origin xyz="0 0 0" rpy="0 0 0" />
-      <geometry>
-        <mesh filename="file://$(find spider_description)/meshes/visual/base_link.STL" />
-      </geometry>
-      <material name="">
-        <color rgba="0.752941176470588 0.752941176470588 0.752941176470588 1" />
-      </material>
-    </visual>
-    <collision>
-      <origin xyz="0 0 0" rpy="0 0 0" />
-      <geometry>
-        <mesh filename="file://$(find spider_description)/meshes/collision/base_link.STL" />
+      <inertia ixx="9.18101041743378E-05" ixy="-1.10969157176021E-06" ixz="-2.07334737671984E-08" iyy="0.000621158029436724" iyz="3.17880975410804E-08" izz="0.000699601373790156" />
+    </inertial>
+    <visual>
+      <origin xyz="0 0 0" rpy="0 0 0" />
+      <geometry>
+        <mesh filename="$(find spider_description)/meshes/visual/base_link.STL" />
+      </geometry>
+      <material name="">
+        <color rgba="0.752941176470588 0.752941176470588 0.752941176470588 1" />
+      </material>
+    </visual>
+    <collision>
+      <origin xyz="0 0 0" rpy="0 0 0" />
+      <geometry>
+        <mesh filename="$(find spider_description)/meshes/collision/base_link.STL" />
       </geometry>
     </collision>
@@ -30,21 +34,21 @@
   <link name="RL1_coxa">
     <inertial>
-      <origin xyz="-0.00349163844394274 0.017230005966643 0.0244390511872048" rpy="0 0 0" />
+      <origin xyz="-0.00349163844394271 0.017230005966643 0.0244390511872048" rpy="0 0 0" />
       <mass value="0.0118214531865819" />
-      <inertia ixx="1.54720054808557E-06" ixy="-3.57557713352019E-08" ixz="-4.02762646820984E-08" iyy="1.03828147386784E-06" iyz="-8.80078006023742E-10" izz="1.47258288978444E-06" />
-    </inertial>
-    <visual>
-      <origin xyz="0 0 0" rpy="0 0 0" />
-      <geometry>
-        <mesh filename="file://$(find spider_description)/meshes/visual/RL1_coxa.STL" />
-      </geometry>
-      <material name="">
-        <color rgba="0.752941176470588 0.752941176470588 0.752941176470588 1" />
-      </material>
-    </visual>
-    <collision>
-      <origin xyz="0 0 0" rpy="0 0 0" />
-      <geometry>
-        <mesh filename="file://$(find spider_description)/meshes/collision/RL1_coxa.STL" />
+      <inertia ixx="1.54720054808557E-06" ixy="-3.57557713352019E-08" ixz="-4.02762646820984E-08" iyy="1.03828147386784E-06" iyz="-8.80078006023775E-10" izz="1.47258288978444E-06" />
+    </inertial>
+    <visual>
+      <origin xyz="0 0 0" rpy="0 0 0" />
+      <geometry>
+        <mesh filename="$(find spider_description)/meshes/visual/RL1_coxa.STL" />
+      </geometry>
+      <material name="">
+        <color rgba="0.752941176470588 0.752941176470588 0.752941176470588 1" />
+      </material>
+    </visual>
+    <collision>
+      <origin xyz="0 0 0" rpy="0 0 0" />
+      <geometry>
+        <mesh filename="$(find spider_description)/meshes/collision/RL1_coxa.STL" />
       </geometry>
     </collision>
@@ -58,12 +62,12 @@
   <link name="RL1_fumer">
     <inertial>
-      <origin xyz="-0.0264233888332985 -1.38777878078145E-17 -0.00234030420177742" rpy="0 0 0" />
+      <origin xyz="-0.0264233888332985 -2.08166817117217E-17 -0.00234030420177739" rpy="0 0 0" />
       <mass value="0.00732061922605987" />
-      <inertia ixx="1.66034801156123E-06" ixy="-7.94093388050907E-22" ixz="-1.49987503139404E-09" iyy="3.3348950865199E-06" iyz="1.28978137012331E-21" izz="1.8515397312667E-06" />
-    </inertial>
-    <visual>
-      <origin xyz="0 0 0" rpy="0 0 0" />
-      <geometry>
-        <mesh filename="file://$(find spider_description)/meshes/visual/RL1_fumer.STL" />
+      <inertia ixx="1.66034801156123E-06" ixy="-8.99972506457694E-22" ixz="-1.499875031394E-09" iyy="3.3348950865199E-06" iyz="1.31159825877939E-21" izz="1.8515397312667E-06" />
+    </inertial>
+    <visual>
+      <origin xyz="0 0 0" rpy="0 0 0" />
+      <geometry>
+        <mesh filename="$(find spider_description)/meshes/visual/RL1_fumer.STL" />
       </geometry>
       <material name="">
@@ -74,5 +78,5 @@
       <origin xyz="0 0 0" rpy="0 0 0" />
       <geometry>
-        <mesh filename="file://$(find spider_description)/meshes/collision/RL1_fumer.STL" />
+        <mesh filename="$(find spider_description)/meshes/collision/RL1_fumer.STL" />
       </geometry>
     </collision>
@@ -86,21 +90,21 @@
   <link name="RL1_tibia">
     <inertial>
-      <origin xyz="0.00260154713513186 -0.0130975375024425 0.000727426073779153" rpy="0 0 0" />
+      <origin xyz="0.00260154713513185 -0.0130975375024425 0.00072742607377918" rpy="0 0 0" />
       <mass value="0.013123891605465" />
-      <inertia ixx="4.2299662226924E-06" ixy="1.19149413513681E-07" ixz="-1.17548988409946E-08" iyy="7.82194147309099E-07" iyz="-2.83284559215829E-07" izz="4.42455942176531E-06" />
-    </inertial>
-    <visual>
-      <origin xyz="0 0 0" rpy="0 0 0" />
-      <geometry>
-        <mesh filename="file://$(find spider_description)/meshes/visual/RL1_tibia.STL" />
-      </geometry>
-      <material name="">
-        <color rgba="0.752941176470588 0.752941176470588 0.752941176470588 1" />
-      </material>
-    </visual>
-    <collision>
-      <origin xyz="0 0 0" rpy="0 0 0" />
-      <geometry>
-        <mesh filename="file://$(find spider_description)/meshes/collision/RL1_tibia.STL" />
+      <inertia ixx="4.2299662226924E-06" ixy="1.19149413513681E-07" ixz="-1.17548988409948E-08" iyy="7.82194147309099E-07" iyz="-2.83284559215829E-07" izz="4.42455942176531E-06" />
+    </inertial>
+    <visual>
+      <origin xyz="0 0 0" rpy="0 0 0" />
+      <geometry>
+        <mesh filename="$(find spider_description)/meshes/visual/RL1_tibia.STL" />
+      </geometry>
+      <material name="">
+        <color rgba="0.752941176470588 0.752941176470588 0.752941176470588 1" />
+      </material>
+    </visual>
+    <collision>
+      <origin xyz="0 0 0" rpy="0 0 0" />
+      <geometry>
+        <mesh filename="$(find spider_description)/meshes/collision/RL1_tibia.STL" />
       </geometry>
     </collision>
@@ -116,19 +120,19 @@
       <origin xyz="-0.00137410211994941 0.017230005966643 0.024648947347057" rpy="0 0 0" />
       <mass value="0.0118214531865819" />
-      <inertia ixx="1.53973619894474E-06" ixy="-3.56987341340023E-08" ixz="-4.6080725279413E-08" iyy="1.03828147386784E-06" iyz="2.20229478084549E-09" izz="1.48004723892527E-06" />
-    </inertial>
-    <visual>
-      <origin xyz="0 0 0" rpy="0 0 0" />
-      <geometry>
-        <mesh filename="file://$(find spider_description)/meshes/visual/RL2_coxa.STL" />
-      </geometry>
-      <material name="">
-        <color rgba="0.752941176470588 0.752941176470588 0.752941176470588 1" />
-      </material>
-    </visual>
-    <collision>
-      <origin xyz="0 0 0" rpy="0 0 0" />
-      <geometry>
-        <mesh filename="file://$(find spider_description)/meshes/collision/RL2_coxa.STL" />
+      <inertia ixx="1.53973619894474E-06" ixy="-3.56987341340022E-08" ixz="-4.6080725279413E-08" iyy="1.03828147386784E-06" iyz="2.2022947808455E-09" izz="1.48004723892527E-06" />
+    </inertial>
+    <visual>
+      <origin xyz="0 0 0" rpy="0 0 0" />
+      <geometry>
+        <mesh filename="$(find spider_description)/meshes/visual/RL2_coxa.STL" />
+      </geometry>
+      <material name="">
+        <color rgba="0.752941176470588 0.752941176470588 0.752941176470588 1" />
+      </material>
+    </visual>
+    <collision>
+      <origin xyz="0 0 0" rpy="0 0 0" />
+      <geometry>
+        <mesh filename="$(find spider_description)/meshes/collision/RL2_coxa.STL" />
       </geometry>
     </collision>
@@ -144,10 +148,10 @@
       <origin xyz="-0.0264233888332987 6.24500451351651E-17 0.0581596957982228" rpy="0 0 0" />
       <mass value="0.00732061922605988" />
-      <inertia ixx="1.66034801156124E-06" ixy="5.82335151237331E-22" ixz="-1.49987503139389E-09" iyy="3.33489508651991E-06" iyz="3.18774728562622E-22" izz="1.85153973126671E-06" />
-    </inertial>
-    <visual>
-      <origin xyz="0 0 0" rpy="0 0 0" />
-      <geometry>
-        <mesh filename="file://$(find spider_description)/meshes/visual/RL2_fumer.STL" />
+      <inertia ixx="1.66034801156124E-06" ixy="6.88214269644119E-22" ixz="-1.49987503139386E-09" iyy="3.33489508651991E-06" iyz="3.43796942092352E-22" izz="1.85153973126671E-06" />
+    </inertial>
+    <visual>
+      <origin xyz="0 0 0" rpy="0 0 0" />
+      <geometry>
+        <mesh filename="$(find spider_description)/meshes/visual/RL2_fumer.STL" />
       </geometry>
       <material name="">
@@ -158,5 +162,5 @@
       <origin xyz="0 0 0" rpy="0 0 0" />
       <geometry>
-        <mesh filename="file://$(find spider_description)/meshes/collision/RL2_fumer.STL" />
+        <mesh filename="$(find spider_description)/meshes/collision/RL2_fumer.STL" />
       </geometry>
     </collision>
@@ -172,19 +176,19 @@
       <origin xyz="-0.0562495143524853 -0.0130839593275274 -0.00677615060162512" rpy="0 0 0" />
       <mass value="0.013123891605465" />
-      <inertia ixx="4.23019150195768E-06" ixy="7.84253861591576E-08" ixz="1.01977946227722E-09" iyy="7.65338483748999E-07" iyz="-1.6371410447347E-07" izz="4.44118980606013E-06" />
-    </inertial>
-    <visual>
-      <origin xyz="0 0 0" rpy="0 0 0" />
-      <geometry>
-        <mesh filename="file://$(find spider_description)/meshes/visual/RL2_tibia.STL" />
-      </geometry>
-      <material name="">
-        <color rgba="0.752941176470588 0.752941176470588 0.752941176470588 1" />
-      </material>
-    </visual>
-    <collision>
-      <origin xyz="0 0 0" rpy="0 0 0" />
-      <geometry>
-        <mesh filename="file://$(find spider_description)/meshes/collision/RL2_tibia.STL" />
+      <inertia ixx="4.23019150195768E-06" ixy="7.84253861591576E-08" ixz="1.01977946227711E-09" iyy="7.65338483748999E-07" iyz="-1.6371410447347E-07" izz="4.44118980606013E-06" />
+    </inertial>
+    <visual>
+      <origin xyz="0 0 0" rpy="0 0 0" />
+      <geometry>
+        <mesh filename="$(find spider_description)/meshes/visual/RL2_tibia.STL" />
+      </geometry>
+      <material name="">
+        <color rgba="0.752941176470588 0.752941176470588 0.752941176470588 1" />
+      </material>
+    </visual>
+    <collision>
+      <origin xyz="0 0 0" rpy="0 0 0" />
+      <geometry>
+        <mesh filename="$(find spider_description)/meshes/collision/RL2_tibia.STL" />
       </geometry>
     </collision>
@@ -200,19 +204,19 @@
       <origin xyz="0.00349358134474833 0.017230005966643 0.0244387735236787" rpy="0 0 0" />
       <mass value="0.0118214531865818" />
-      <inertia ixx="1.51968642178633E-06" ixy="-3.45709794269535E-08" ixz="-5.40202742068447E-08" iyy="1.03828147386784E-06" iyz="9.17044723735258E-09" izz="1.50009701608367E-06" />
-    </inertial>
-    <visual>
-      <origin xyz="0 0 0" rpy="0 0 0" />
-      <geometry>
-        <mesh filename="file://$(find spider_description)/meshes/visual/RL3_coxa.STL" />
-      </geometry>
-      <material name="">
-        <color rgba="0.752941176470588 0.752941176470588 0.752941176470588 1" />
-      </material>
-    </visual>
-    <collision>
-      <origin xyz="0 0 0" rpy="0 0 0" />
-      <geometry>
-        <mesh filename="file://$(find spider_description)/meshes/collision/RL3_coxa.STL" />
+      <inertia ixx="1.51968642178633E-06" ixy="-3.45709794269535E-08" ixz="-5.40202742068447E-08" iyy="1.03828147386784E-06" iyz="9.17044723735254E-09" izz="1.50009701608367E-06" />
+    </inertial>
+    <visual>
+      <origin xyz="0 0 0" rpy="0 0 0" />
+      <geometry>
+        <mesh filename="$(find spider_description)/meshes/visual/RL3_coxa.STL" />
+      </geometry>
+      <material name="">
+        <color rgba="0.752941176470588 0.752941176470588 0.752941176470588 1" />
+      </material>
+    </visual>
+    <collision>
+      <origin xyz="0 0 0" rpy="0 0 0" />
+      <geometry>
+        <mesh filename="$(find spider_description)/meshes/collision/RL3_coxa.STL" />
       </geometry>
     </collision>
@@ -228,10 +232,10 @@
       <origin xyz="-0.0264233888332993 -3.12250225675825E-16 0.118659695798224" rpy="0 0 0" />
       <mass value="0.00732061922605988" />
-      <inertia ixx="1.66034801156124E-06" ixy="-1.05879118406788E-22" ixz="-1.49987503139562E-09" iyy="3.33489508651991E-06" iyz="-7.61987364388377E-23" izz="1.85153973126671E-06" />
-    </inertial>
-    <visual>
-      <origin xyz="0 0 0" rpy="0 0 0" />
-      <geometry>
-        <mesh filename="file://$(find spider_description)/meshes/visual/RL3_fumer.STL" />
+      <inertia ixx="1.66034801156124E-06" ixy="-5.29395592033938E-23" ixz="-1.49987503139564E-09" iyy="3.33489508651991E-06" iyz="-7.52681582497153E-23" izz="1.85153973126671E-06" />
+    </inertial>
+    <visual>
+      <origin xyz="0 0 0" rpy="0 0 0" />
+      <geometry>
+        <mesh filename="$(find spider_description)/meshes/visual/RL3_fumer.STL" />
       </geometry>
       <material name="">
@@ -242,5 +246,5 @@
       <origin xyz="0 0 0" rpy="0 0 0" />
       <geometry>
-        <mesh filename="file://$(find spider_description)/meshes/collision/RL3_fumer.STL" />
+        <mesh filename="$(find spider_description)/meshes/collision/RL3_fumer.STL" />
       </geometry>
     </collision>
@@ -254,21 +258,21 @@
   <link name="RL3_tibia">
     <inertial>
-      <origin xyz="-0.118005534421714 -0.0130894519462948 0.00839605198202775" rpy="0 0 0" />
+      <origin xyz="-0.118005534421714 -0.0130894519462948 0.00839605198202772" rpy="0 0 0" />
       <mass value="0.013123891605465" />
-      <inertia ixx="4.23878065273637E-06" ixy="4.20082265127764E-08" ixz="4.18757931219035E-08" iyy="7.691544615372E-07" iyz="-2.12494160023349E-07" izz="4.42878467749324E-06" />
-    </inertial>
-    <visual>
-      <origin xyz="0 0 0" rpy="0 0 0" />
-      <geometry>
-        <mesh filename="file://$(find spider_description)/meshes/visual/RL3_tibia.STL" />
-      </geometry>
-      <material name="">
-        <color rgba="0.752941176470588 0.752941176470588 0.752941176470588 1" />
-      </material>
-    </visual>
-    <collision>
-      <origin xyz="0 0 0" rpy="0 0 0" />
-      <geometry>
-        <mesh filename="file://$(find spider_description)/meshes/collision/RL3_tibia.STL" />
+      <inertia ixx="4.23878065273637E-06" ixy="4.20082265127764E-08" ixz="4.18757931219034E-08" iyy="7.69154461537199E-07" iyz="-2.12494160023349E-07" izz="4.42878467749323E-06" />
+    </inertial>
+    <visual>
+      <origin xyz="0 0 0" rpy="0 0 0" />
+      <geometry>
+        <mesh filename="$(find spider_description)/meshes/visual/RL3_tibia.STL" />
+      </geometry>
+      <material name="">
+        <color rgba="0.752941176470588 0.752941176470588 0.752941176470588 1" />
+      </material>
+    </visual>
+    <collision>
+      <origin xyz="0 0 0" rpy="0 0 0" />
+      <geometry>
+        <mesh filename="$(find spider_description)/meshes/collision/RL3_tibia.STL" />
       </geometry>
     </collision>
@@ -282,5 +286,5 @@
   <link name="RL4_coxa">
     <inertial>
-      <origin xyz="0.000221643372700031 0.0172339889705058 0.0247738629223978" rpy="0 0 0" />
+      <origin xyz="0.000221643372700024 0.0172339889705058 0.0247738629223978" rpy="0 0 0" />
       <mass value="0.011831113051677" />
       <inertia ixx="1.51589381883954E-06" ixy="3.36933681099745E-08" ixz="5.44221588671393E-08" iyy="1.03946591481982E-06" iyz="1.04055511028782E-08" izz="1.50574484630922E-06" />
@@ -289,14 +293,14 @@
       <origin xyz="0 0 0" rpy="0 0 0" />
       <geometry>
-        <mesh filename="file://$(find spider_description)/meshes/visual/RL4_coxa.STL" />
-      </geometry>
-      <material name="">
-        <color rgba="0.752941176470588 0.752941176470588 0.752941176470588 1" />
-      </material>
-    </visual>
-    <collision>
-      <origin xyz="0 0 0" rpy="0 0 0" />
-      <geometry>
-        <mesh filename="file://$(find spider_description)/meshes/collision/RL4_coxa.STL" />
+        <mesh filename="$(find spider_description)/meshes/visual/RL4_coxa.STL" />
+      </geometry>
+      <material name="">
+        <color rgba="0.752941176470588 0.752941176470588 0.752941176470588 1" />
+      </material>
+    </visual>
+    <collision>
+      <origin xyz="0 0 0" rpy="0 0 0" />
+      <geometry>
+        <mesh filename="$(find spider_description)/meshes/collision/RL4_coxa.STL" />
       </geometry>
     </collision>
@@ -310,12 +314,12 @@
   <link name="RL4_fumer">
     <inertial>
-      <origin xyz="-0.0264233888332989 1.38777878078145E-17 -0.176940304201777" rpy="0 0 0" />
+      <origin xyz="-0.0264233888332989 6.93889390390723E-18 -0.176940304201777" rpy="0 0 0" />
       <mass value="0.00732061922605987" />
-      <inertia ixx="1.66034801156123E-06" ixy="5.29395592033938E-22" ixz="-1.49987503139488E-09" iyy="3.3348950865199E-06" iyz="1.40101077504865E-22" izz="1.85153973126671E-06" />
-    </inertial>
-    <visual>
-      <origin xyz="0 0 0" rpy="0 0 0" />
-      <geometry>
-        <mesh filename="file://$(find spider_description)/meshes/visual/RL4_fumer.STL" />
+      <inertia ixx="1.66034801156123E-06" ixy="5.29395592033938E-22" ixz="-1.49987503139487E-09" iyy="3.3348950865199E-06" iyz="1.10684466970948E-22" izz="1.85153973126671E-06" />
+    </inertial>
+    <visual>
+      <origin xyz="0 0 0" rpy="0 0 0" />
+      <geometry>
+        <mesh filename="$(find spider_description)/meshes/visual/RL4_fumer.STL" />
       </geometry>
       <material name="">
@@ -326,5 +330,5 @@
       <origin xyz="0 0 0" rpy="0 0 0" />
       <geometry>
-        <mesh filename="file://$(find spider_description)/meshes/collision/RL4_fumer.STL" />
+        <mesh filename="$(find spider_description)/meshes/collision/RL4_fumer.STL" />
       </geometry>
     </collision>
@@ -338,21 +342,21 @@
   <link name="RL4_tibia">
     <inertial>
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
Commit message: final_v1_controlling-perfectlty

File: spider_description/urdf/spider_description.xacro (robot description, xacro)
@@ -114,5 +114,5 @@
     <parent link="RL1_fumer" />
     <child link="RL1_tibia" />
-    <axis xyz="0.976555650922224 0 0.215265093900221" />
+    <axis xyz="-0.976555650922224 0 -0.215265093900221" />
   </joint>
   <link name="RL2_coxa">
@@ -198,5 +198,5 @@
     <parent link="RL2_fumer" />
     <child link="RL2_tibia" />
-    <axis xyz="0.991465481571485 0 0.130369470552824" />
+    <axis xyz="-0.991465481571485 0 -0.130369470552824" />
   </joint>
   <link name="RL3_coxa">
@@ -282,5 +282,5 @@
     <parent link="RL3_fumer" />
     <child link="RL3_tibia" />
-    <axis xyz="0.997760486341758 0 -0.0668880549504799" />
+    <axis xyz="-0.997760486341758 0 0.0668880549504799" />
   </joint>
   <link name="RL4_coxa">
@@ -338,5 +338,5 @@
     <parent link="RL4_coxa" />
     <child link="RL4_fumer" />
-    <axis xyz="0 0 1" />
+    <axis xyz="0 0 -1" />
   </joint>
   <link name="RL4_tibia">
@@ -366,5 +366,5 @@
     <parent link="RL4_fumer" />
     <child link="RL4_tibia" />
-    <axis xyz="0.994460811195995 0 0.105108015847522" />
+    <axis xyz="-0.994460811195995 0 -0.105108015847522" />
   </joint>
   <link name="LL1_coxa">
@@ -394,5 +394,5 @@
     <parent link="base_link" />
     <child link="LL1_coxa" />
-    <axis xyz="0 1 0" />
+    <axis xyz="0 -1 0" />
   </joint>
   <link name="LL1_fumer">
@@ -422,5 +422,5 @@
     <parent link="LL1_coxa" />
     <child link="LL1_fumer" />
-    <axis xyz="0 0 1" />
+    <axis xyz="0 0 -1" />
   </joint>
   <link name="LL1_tibia">
@@ -478,5 +478,5 @@
     <parent link="base_link" />
     <child link="LL2_coxa" />
-    <axis xyz="0 1 0" />
+    <axis xyz="0 -1 0" />
   </joint>
   <link name="LL2_fumer">
@@ -506,5 +506,5 @@
     <parent link="LL2_coxa" />
     <child link="LL2_fumer" />
-    <axis xyz="0 0 1" />
+    <axis xyz="0 0 -1" />
   </joint>
   <link name="LL2_tibia">
@@ -562,5 +562,5 @@
     <parent link="base_link" />
     <child link="LL3_coxa" />
-    <axis xyz="0 1 0" />
+    <axis xyz="0 -1 0" />
   </joint>
   <link name="LL3_fumer">
@@ -590,5 +590,5 @@
     <parent link="LL3_coxa" />
     <child link="LL3_fumer" />
-    <axis xyz="0 0 1" />
+    <axis xyz="0 0 -1" />
   </joint>
   <link name="LL3_tibia">
@@ -646,5 +646,5 @@
     <parent link="base_link" />
     <child link="LL4_coxa" />
-    <axis xyz="0 1 0" />
+    <axis xyz="0 -1 0" />
   </joint>
   <link name="LL4_fumer">
